Commit message: update ranger_mini_v3 model and dae

File: ranger_mini/ranger_mini_v3/urdf/ranger_mini.xacro (robot description, xacro)
@@ -1,55 +1,189 @@
-<?xml version="1.0"?>
-<robot name="ranger_mini_v2"
-    xmlns:xacro="http://ros.org/wiki/xacro">
-    <xacro:include filename="$(find ranger_mini_v2)/urdf/ranger_l.xacro" />
-    <xacro:include filename="$(find ranger_mini_v2)/urdf/ranger_r.xacro" />
-    <!-- Variables -->
-    <xacro:property name="M_PI" value="3.14159"/>
-    <!-- Vehicle Geometries -->
-    <xacro:property name="base_x_size" value="1.0" />
-    <xacro:property name="base_y_size" value="0.380000" />
-    <xacro:property name="base_z_size" value="0.210000" />
-    <xacro:property name="wheelbase" value="0.498" />
-    <xacro:property name="track" value="0.58306" />
-    <xacro:property name="wheel_vertical_offset" value="-0.0702" />
-    <xacro:property name="wheel_length" value="1.1653e-01" />
-    <xacro:property name="wheel_radius" value="1.6459e-01" />
-    <!-- Base link -->
-    <link name="base_link">
-        <visual>
-            <origin xyz="0 0 0" rpy="1.57 0 3.14 " />
+<?xml version="1.0" encoding="utf-8"?>
+<robot name="ranger_mini_v3"  xmlns:xacro="http://ros.org/wiki/xacro">
+  <link
+    name="base_link">
+    <inertial>
+      <origin
+        xyz="-0.0242698272228022 -0.0030308024613212 0.0544267444673498"
+        rpy="0 0 0" />
+      <mass
+        value="10" />
+      <inertia ixx="0.1354" ixy="0.0" ixz="0.0" iyy="0.2417" iyz="0.0" izz="0.3085"/>
+    </inertial>
+    <visual>
+      <origin
+        xyz="0 0 0.0"
+        rpy="0 0 0" />
+      <geometry>
+        <mesh
+          filename="package://ranger_mini_v3/meshes/ranger_base.dae" scale="1000 1000 1000" />
+      </geometry>
+      <material
+        name="">
+        <color
+          rgba="0.792156862745098 0.819607843137255 0.933333333333333 1" />
+      </material>
+    </visual>
+        <collision>
+            <origin xyz="0 0 -0.1" rpy="0 0 0" />
             <geometry>
-                <mesh filename="package://ranger_mini_v2/meshes/ranger_base.dae" />
-            </geometry>
-        </visual>
-        <collision>
-            <origin xyz="0 0 0.008" rpy="0 0 0" />
-            <geometry>
-                <box size="1 1 1"/>
+                <box size="0.5 0.35 0.2"/>
             </geometry>
         </collision>
-        <collision>
-            <origin xyz="0 0 0" rpy="0 0 0" />
-            <geometry>
-                <box size="1 1 1"/>
-            </geometry>
-        </collision>
-    </link>
+   </link>
+   <link
+    name="fr_steering_wheel_link">
+    <inertial>
+      <origin
+        xyz="1.8493E-05 1.2713E-06 0.043679"
+        rpy="0 0 0" />
+      <mass
+        value="1" />
+      <inertia
+        ixx="0.0063625"
+        ixy="-1.0581E-07"
+        ixz="-4.0831E-07"
+        iyy="0.006363"
+        iyz="-3.4944E-08"
+        izz="0.010465" />
+    </inertial>
+    <visual>
+      <origin
+        xyz="0 0 0"
+        rpy="0 0 0" />
+      <geometry>
+        <mesh filename="package://ranger_mini_v3/meshes/steering_wheel.dae" scale="10 10 10"/>
+      </geometry>
+      <material
+        name="">
+        <color
+          rgba="0.79216 0.81961 0.93333 1" />
+      </material>
+    </visual>
+    <collision>
+      <origin
+        xyz="0 0 0"
+        rpy="0 0 0" />
+      <geometry>
+        <!-- <mesh
+          filename="package://ranger_mini_v3/meshes/ranger_mini_v3_wheel_right.dae" /> -->
+          <cylinder radius="0.001" length="0.001"/>
+      </geometry>
+    </collision>
+  </link>
+  <joint
+    name="fr_steering_joint"
+    type="revolute">
+    <origin
+      xyz="0.25 -0.19 -0.1"
+      rpy="0 0 0" />
+    <parent
+      link="base_link" />
+    <child
+      link="fr_steering_wheel_link" />
+    <axis
+      xyz="0 0 -1" />
+    <limit effort="5" velocity="6.28"  lower="-2.1" upper="2.1" />
+  </joint>
+  <link name="fr_wheel_link">
+      <inertial>
+          <mass value="8" />
+          <origin xyz="0 0 0" />
+          <inertia ixx="0.02047" ixy="0.0" ixz="0.0" iyy="0.02047" iyz="0.0" izz="0.0324"/>
+          </inertial>
+      <visual>
+          <origin xyz="0 0 0" rpy="3.14 0 0" />
+          <geometry>
+            <mesh filename="package://ranger_mini_v3/meshes/wheel_v3.dae" scale="10 10 10"/>
+          </geometry>
+      </visual>
+      <collision>
+          <origin xyz="0 0 -0.005" rpy="1.57 0 0" />
+          <geometry>
+              <cylinder length="0.08" radius="0.09" />
+          </geometry>
+                <contact>
+                    <ode>
+                  <min_depth>0.001</min_depth>
+                    </ode>
+              </contact>
+      </collision>
+  </link>
+        <joint name="fr_wheel" type="continuous">
+            <origin xyz="0.0 0.0 -0.12" rpy="0 0 0" />
+            <parent link="fr_steering_wheel_link"/>
+            <child link="fr_wheel_link"/>
+            <axis xyz="0 1 0" rpy="0 0 0" />
+        </joint>
+  <link
+    name="fl_steering_wheel_link">
+    <inertial>
+      <origin
+        xyz="-0.0017956 -9.6304E-08 0.043642"
+        rpy="0 0 0" />
+      <mass
+        value="1" />
+      <inertia
+        ixx="0.0063695"
+        ixy="-2.1067E-08"
+        ixz="-0.00016867"
+        iyy="0.006363"
+        iyz="-1.0301E-08"
+        izz="0.010458" />
+    </inertial>
+    <visual>
+      <origin
+        xyz="0 0 0"
+        rpy="0 0 3.14" />
+      <geometry>
+        <mesh filename="package://ranger_mini_v3/meshes/steering_wheel.dae" scale="10 10 10"/>
+      </geometry>
+      <material
+        name="">
+        <color
+          rgba="0.79216 0.81961 0.93333 1" />
+      </material>
+    </visual>
+    <collision>
+      <origin
+        xyz="0 0 0"
+        rpy="0 0 0" />
+      <geometry>
+        <!-- <mesh
+          filename="package://ranger_mini_v3/meshes/ranger_mini_v3_wheel.dae" /> -->
+        <cylinder radius="0.001" length="0.001"/>
+      </geometry>
+    </collision>
+  </link>
+   <joint
+    name="fl_steering_joint"
+    type="revolute">
+    <origin
+      xyz="0.25 0.19 -0.1"
+      rpy="0 0 0" />
+    <parent
+      link="base_link" />
+    <child
+      link="fl_steering_wheel_link" />
+    <axis
+      xyz="0 0 -1" />
+        <limit effort="5" velocity="6.28"  lower="-2.1" upper="2.1" />
+  </joint>
         <link name="fl_wheel_link">
             <inertial>
                 <mass value="8" />
                 <origin xyz="0 0 0" />
-                <inertia ixx="0.1171" ixy="0" ixz="0" iyy="0.1361" iyz="0" izz="0.1171" />
+                <inertia ixx="0.02047" ixy="0.0" ixz="0.0" iyy="0.02047" iyz="0.0" izz="0.0324"/>
             </inertial>
             <visual>
-                <origin xyz="0.23 -0.2 0.1" rpy="1.57 0 0" />
-                <geometry>
-                    <mesh filename="package://ranger_mini_v2/meshes/fr.dae" />
+                <origin xyz="0 0 0" rpy="0 0 0" />
+                <geometry>
+                <mesh filename="package://ranger_mini_v3/meshes/wheel_v3.dae" scale="10 10 10"/>
                 </geometry>
             </visual>
             <collision>
-                <origin xyz="0 0 0" rpy="0 0 0" />
-                <geometry>
-                    <cylinder length="0.1" radius="0.1" />
+                <origin xyz="0 0 -0.005" rpy="1.57 0 0" />
+                <geometry>
+                    <cylinder length="0.08" radius="0.09" />
                 </geometry>
                      <contact>
@@ -61,55 +195,79 @@
         </link>
         <joint name="fl_wheel" type="continuous">
-            <origin xyz="0.23 0.206 -0.1" rpy="0 0 0" />
-            <parent link="base_link"/>
+            <origin xyz="0.0 0.0 -0.12" rpy="0 0 0" />
+            <parent link="fl_steering_wheel_link"/>
             <child link="fl_wheel_link"/>
-            <axis xyz="0 -1 0" rpy="0 0 0" />
+            <axis xyz="0 1 0" rpy="0 0 0" />
         </joint>
-        <link name="fr_wheel_link">
-            <inertial>
-                <mass value="8" />
-                <origin xyz="0 0 0" />
-                <inertia ixx="0.1171" ixy="0" ixz="0" iyy="0.1361" iyz="0" izz="0.1171" />
-            </inertial>
-            <visual>
-                <origin xyz="0.23 0.2 0.1" rpy="1.57 0 0" />
-                <geometry>
-                    <mesh filename="package://ranger_mini_v2/meshes/fl.dae" />
-                </geometry>
-            </visual>
-            <collision>
-                <origin xyz="0 0 0" rpy="0 0 0" />
-                <geometry>
-                    <cylinder length="0.1" radius="0.1" />
-                </geometry>
-                     <contact>
-                         <ode>
-                        <min_depth>0.001</min_depth>
-                         </ode>
-                    </contact>
-            </collision>
-        </link>
-        <joint name="fr_wheel" type="continuous">
-            <origin xyz="0.23 -0.206 -0.1" rpy="0 0 0" />
-            <parent link="base_link"/>
-            <child link="fr_wheel_link"/>
-            <axis xyz="0 -1 0" rpy="0 0 0" />
-        </joint>
+ <link
+    name="rl_steering_wheel_link">
+    <inertial>
+      <origin
+        xyz="-0.00017093 6.1255E-08 0.043678"
+        rpy="0 0 0" />
+      <mass
+        value="1" />
+      <inertia
+        ixx="0.0063627"
+        ixy="-2.1069E-08"
+        ixz="-1.587E-05"
+        iyy="0.006363"
+        iyz="9.3201E-09"
+        izz="0.010465" />
+    </inertial>
+    <visual>
+      <origin
+        xyz="0 0 0"
+        rpy="0 0 3.14" />
+      <geometry>
+        <mesh filename="package://ranger_mini_v3/meshes/steering_wheel.dae" scale="10 10 10"/>
+      </geometry>
+      <material
+        name="">
+        <color
+          rgba="0.79216 0.81961 0.93333 1" />
+      </material>
+    </visual>
+    <collision>
+      <origin
+        xyz="0 0 0"
+        rpy="0 0 0" />
+      <geometry>
+        <!-- <mesh
+          filename="package://ranger_mini_v3/meshes/ranger_mini_v3_wheel_right.dae" /> -->
+        <cylinder radius="0.001" length="0.001"/>
+      </geometry>
+    </collision>
+  </link>
+  <joint
+    name="rl_steering_joint"
+    type="revolute">
+    <origin
+      xyz="-0.25 0.19 -0.1"
+      rpy="0 0 0" />
+    <parent
+      link="base_link" />
+    <child
+      link="rl_steering_wheel_link" />
+    <axis
+      xyz="0 0 -1" />
+        <limit effort="5" velocity="6.28"  lower="-2.1" upper="2.1" />
+  </joint>
         <link name="rl_wheel_link">
             <inertial>
                 <mass value="8" />
                 <origin xyz="0 0 0" />
-                <inertia ixx="0.1171" ixy="0" ixz="0" iyy="0.1361" iyz="0" izz="0.1171" />
+                <inertia ixx="0.02047" ixy="0.0" ixz="0.0" iyy="0.02047" iyz="0.0" izz="0.0324"/>
             </inertial>
             <visual>
-                <origin xyz="0.23 -0.2 0.1" rpy="1.57 0 0" />
-                <geometry>
-                    <mesh filename="package://ranger_mini_v2/meshes/fr.dae" />
+                <origin xyz="0 0 0" rpy="0 0 0" />
+                <geometry>
+                  <mesh filename="package://ranger_mini_v3/meshes/wheel_v3.dae" scale="10 10 10"/>
                 </geometry>
             </visual>
             <collision>
-                <origin xyz="0 0 0" rpy="0 0 0" />
-                <geometry>
-                    <cylinder length="0.1" radius="0.1" />
+                <origin xyz="0.00 0.00 -0.005" rpy="1.57 0 0" />
+                <geometry>
+                    <cylinder length="0.08" radius="0.09" />
                 </geometry>
                      <contact>
@@ -121,25 +279,53 @@
         </link>
         <joint name="rl_wheel" type="continuous">
-            <origin xyz="-0.23 0.206 -0.1" rpy="0 0 0" />
-            <parent link="base_link"/>
+            <origin xyz="0.0 0.0 -0.12 " rpy="0 0 0" />
+            <parent link="rl_steering_wheel_link"/>
             <child link="rl_wheel_link"/>
-            <axis xyz="0 -1 0" rpy="0 0 0" />
+            <axis xyz="0 1 0" rpy="0 0 0" />
         </joint>
-        <link name="rr_wheel_link">
+   <link name="rr_steering_wheel_link">
+        <inertial>
+            <origin xyz="0.0 0.0 0.0"/>
+            <mass value="1"/>
+            <inertia ixx="0.01" ixy="0.0" ixz="0.0" iyy="0.01" iyz="0.0" izz="0.01"/>
+        </inertial>
+        <visual>
+          <origin
+            xyz="0 0 0"
+            rpy="0 0 0" />
+          <geometry>
+            <mesh filename="package://ranger_mini_v3/meshes/steering_wheel.dae" scale="10 10 10"/>
+          </geometry>
+        </visual>
+        <collision>
+            <origin  xyz="0 0 0" rpy="0 0 0" />
+                    <geometry>
+                <cylinder radius="0.001" length="0.001"/>
+            </geometry>
+        </collision>
+    </link>
+    <joint name="rr_steering_joint" type="revolute">
+        <origin xyz="-0.23 -0.206 -0.1" rpy="0 0 0" />
+        <parent link="base_link"/>
+        <child link="rr_steering_wheel_link"/>
+        <axis xyz="0 0 -1" rpy="0 0 0" />
+        <limit effort="5" velocity="6.28"  lower="-2.1" upper="2.1" />
+    </joint>
+       <link name="rr_wheel_link">
             <inertial>
                 <mass value="8" />
                 <origin xyz="0 0 0" />
-                <inertia ixx="0.1171" ixy="0" ixz="0" iyy="0.1361" iyz="0" izz="0.1171" />
+                <inertia ixx="0.02047" ixy="0.0" ixz="0.0" iyy="0.02047" iyz="0.0" izz="0.0324"/>
             </inertial>
             <visual>
-                <origin xyz="0.23 0.2 0.1" rpy="1.57 0 0" />
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
File: ranger_mini/ranger_mini_v3_gazebo/xacro/ranger_mini_gazebo.xacro (robot description, xacro)
@@ -14,8 +14,8 @@
       <origin
         xyz="0 0 0.0"
-        rpy="3.14 0 0" />
+        rpy="0 0 0" />
       <geometry>
         <mesh
-          filename="package://ranger_mini_v3/meshes/ranger_mini3.dae" />
+          filename="package://ranger_mini_v3/meshes/ranger_base.dae" scale="1000 1000 1000" />
       </geometry>
       <material
@@ -50,9 +50,8 @@
     <visual>
       <origin
-        xyz="-0.248 -0.113 0.155"
-        rpy="1.57 0 3.14" />
-      <geometry>
-        <mesh
-          filename="package://ranger_mini_v3/meshes/ranger_mini_v3_wheel_right.dae" />
+        xyz="0 0 0"
+        rpy="0 0 0" />
+      <geometry>
+        <mesh filename="package://ranger_mini_v3/meshes/steering_wheel.dae" scale="10 10 10"/>
       </geometry>
       <material
@@ -94,7 +93,7 @@
                 </inertial>
             <visual>
-                <origin xyz="0 0 0" rpy="1.57 0 0" />
-                <geometry>
-                    <cylinder length="0.01" radius="0.01" />
+                <origin xyz="0 0 0" rpy="3.14 0 0" />
+                <geometry>
+                <mesh filename="package://ranger_mini_v3/meshes/wheel_v3.dae" scale="10 10 10"/>
                 </geometry>
             </visual>
@@ -135,9 +134,8 @@
     <visual>
       <origin
-        xyz="-0.248 -0.125 -0.192"
-        rpy="1.57 0.0 3.14" />
-      <geometry>
-        <mesh
-          filename="package://ranger_mini_v3/meshes/ranger_mini_v3_wheel.dae" />
+        xyz="0 0 0"
+        rpy="0 0 3.14" />
+      <geometry>
+        <mesh filename="package://ranger_mini_v3/meshes/steering_wheel.dae" scale="10 10 10"/>
       </geometry>
       <material
@@ -179,11 +177,11 @@
             </inertial>
             <visual>
-                <origin xyz="0 0 0" rpy="1.57 0 0" />
-                <geometry>
-                    <cylinder length="0.01" radius="0.01" />
+                <origin xyz="0 0 0" rpy="0 0 0" />
+                <geometry>
+                  <mesh filename="package://ranger_mini_v3/meshes/wheel_v3.dae" scale="10 10 10"/>
                 </geometry>
             </visual>
             <collision>
-                <origin xyz="0 0 0" rpy="1.57 0 0" />
+                <origin xyz="0 0 -0.005" rpy="1.57 0 0" />
                 <geometry>
                     <cylinder length="0.08" radius="0.09" />
@@ -220,9 +218,8 @@
     <visual>
        <origin
-        xyz="-0.241 -0.11 0.155"
-        rpy="1.57 0 3.14" />
-      <geometry>
-        <mesh
-          filename="package://ranger_mini_v3/meshes/ranger_mini_v3_wheel_right.dae" />
+        xyz="0 0 0"
+        rpy="0 0 3.14" />
+      <geometry>
+        <mesh filename="package://ranger_mini_v3/meshes/steering_wheel.dae" scale="10 10 10"/>
       </geometry>
       <material
@@ -264,11 +261,11 @@
             </inertial>
             <visual>
-                <origin xyz="0 0 0" rpy="1.57 0 0" />
-                <geometry>
-                    <cylinder length="0.01" radius="0.01" />
+                <origin xyz="0 0 0" rpy="0 0 0" />
+                <geometry>
+                  <mesh filename="package://ranger_mini_v3/meshes/wheel_v3.dae" scale="10 10 10"/>
                 </geometry>
             </visual>
             <collision>
-                <origin xyz="0.005 0.005 -0.005" rpy="1.57 0 0" />
+                <origin xyz="0.00 0.00 -0.005" rpy="1.57 0 0" />
                 <geometry>
                     <cylinder length="0.08" radius="0.09" />
@@ -294,7 +291,7 @@
         </inertial>
         <visual>
-            <origin  xyz="-0.262 -0.095 0.155" rpy="1.57 0 3.14 " />
+            <origin  xyz="0 0 0" rpy="0 0 0" />
             <geometry>
-                    <mesh filename="package://ranger_mini_v3/meshes/ranger_mini_v3_wheel_right.dae" />
+            <mesh filename="package://ranger_mini_v3/meshes/steering_wheel.dae" scale="10 10 10"/>
             </geometry>
         </visual>
@@ -320,11 +317,11 @@
             </inertial>
             <visual>
-                <origin xyz="0.0 0.0 0.0" rpy="1.57 0 0" />
-                <geometry>
-                    <cylinder length="0.01" radius="0.01" />
+                <origin xyz="0.0 0.0 0.0" rpy="3.14 0 0" />
+                <geometry>
+                    <mesh filename="package://ranger_mini_v3/meshes/wheel_v3.dae" scale="10 10 10"/>
                 </geometry>
             </visual>
             <collision>
-                <origin xyz="-0.015 0.02 -0.005" rpy="1.57 0 0" />
+                <origin xyz=" 0 0 -0.005" rpy="1.57 0 0" />
                 <geometry>
                     <cylinder length="0.08" radius="0.09" />
