Commit message: fixed scout_mini model

File: scout/scout_description/urdf/mini.xacro (robot description, xacro)
@@ -60,9 +60,12 @@
                 rpy="0 0 0" />
             <mass
-                value="10" />
+                value="5" />
             <inertia
-                ixx="0.1083" ixy="0" ixz="0"
-                iyy="0.15"   iyz="0"
-                izz="0.1083"/>
+                ixx="0.054166666667"
+                ixy="0"
+                ixz="0"
+                iyy="0.075"
+                iyz="0"
+                izz="0.054166666667"/>
             </inertial>
         <visual>
@@ -171,4 +174,5 @@
         <child link="camera_link" />
     </joint>
+<!--
     <link name="inertial_link">
         <inertial>
@@ -182,5 +186,5 @@
         <parent link="base_link" />
         <child link="inertial_link" />
-    </joint>
+    </joint> -->
     <!-- For testing, hang the robot up in the air -->
     <!-- <link name="world" />

File: scout/scout_description/urdf/scout_mini.xacro (robot description, xacro)
@@ -17,4 +17,6 @@
    <xacro:property name="track" value="0.4563536" />
    <xacro:property name="wheel_vertical_offset" value="-0.077" />
+    <xacro:property name="wheel_diameter" value="0.16" />
+    <xacro:property name="wheel_width" value="0.084" />
 <!--    <xacro:property name="track" value="0.3426" />
     <xacro:property name="wheelbase" value="0.3181"/>
@@ -85,15 +87,27 @@
     <!-- wheel labeled from 0 to 3, conter-clockwise, starting from front right wheel -->
     <!-- motor 1 and 2 (left side) are mechanically installed in a reversed direction -->
-    <xacro:scout_mini_wheel_1 wheel_prefix="rear_right">
-        <origin xyz="${wheelbase/2} ${-track/2} ${wheel_vertical_offset}" rpy="0 1.57 0" />
+    <xacro:scout_mini_wheel_1 wheel_prefix="front_left" wheel_diameter="${wheel_diameter}" wheel_width="${wheel_width}">
+    <!--<origin
+            xyz="0 0 0"
+            rpy="0 0 0" />-->
+        <origin xyz="${wheelbase/2} ${track/2} ${wheel_vertical_offset}" rpy="-1.57 0 0" />
     </xacro:scout_mini_wheel_1>
-    <xacro:scout_mini_wheel_2 wheel_prefix="front_right">
-        <origin xyz="${wheelbase/2} ${track/2} ${wheel_vertical_offset}" rpy="0 1.57 0" />
+    <xacro:scout_mini_wheel_2 wheel_prefix="rear_left" wheel_diameter="${wheel_diameter}" wheel_width="${wheel_width}">
+    <!--<origin
+            xyz="0 0 0"
+            rpy="0 0 0" />-->
+        <origin xyz="${-wheelbase/2} ${track/2} ${wheel_vertical_offset}" rpy="-1.57 0 0" />
     </xacro:scout_mini_wheel_2>
-    <xacro:scout_mini_wheel_3 wheel_prefix="front_left">
-        <origin xyz="${-wheelbase/2} ${track/2} ${wheel_vertical_offset}" rpy="0 -1.57 0" />
+    <xacro:scout_mini_wheel_3 wheel_prefix="front_right" wheel_diameter="${wheel_diameter}" wheel_width="${wheel_width}">
+    <!--<origin
+            xyz="0 0 0"
+            rpy="0 0 0" />-->
+        <origin xyz="${wheelbase/2} ${-track/2} ${wheel_vertical_offset+0.001}" rpy="1.57 0 0" />
     </xacro:scout_mini_wheel_3>
-    <xacro:scout_mini_wheel_4 wheel_prefix="rear_left">
-        <origin xyz="${-wheelbase/2} ${-track/2} ${wheel_vertical_offset}" rpy="0 -1.57 0" />
+    <xacro:scout_mini_wheel_4 wheel_prefix="rear_right" wheel_diameter="${wheel_diameter}" wheel_width="${wheel_width}">
+    <!--<origin
+           xyz="0 0 0"
+           rpy="0 0 0" />-->
+        <origin xyz="${-wheelbase/2} ${-track/2} ${wheel_vertical_offset+0.001}" rpy="1.57 0 0" />
     </xacro:scout_mini_wheel_4>
     <!-- Additional definitions -->

File: scout/scout_description/urdf/scout_mini_wheel_2.xacro (robot description, xacro)
@@ -59,7 +59,7 @@
                 rpy="0 0 0" />
               <geometry>
-                <mesh
-                  filename="package://scout_description/meshes/wheel.dae" />
-                  <!-- <cylinder radius="0.08" length="0.084"/> -->
+                <!-- <mesh
+                  filename="package://scout_description/meshes/wheel.dae" /> -->
+                  <cylinder radius="0.08" length="0.084"/>
               </geometry>
             </collision>

File: scout/scout_description/urdf/scout_mini_wheel_3.xacro (robot description, xacro)
@@ -59,7 +59,7 @@
                 rpy="0 0 0" />
               <geometry>
-                <mesh
-                  filename="package://scout_description/meshes/wheel.dae" />
-                  <!-- <cylinder radius="0.08" length="0.084"/> -->
+                <!-- <mesh
+                  filename="package://scout_description/meshes/wheel.dae" /> -->
+                  <cylinder radius="0.08" length="0.084"/>
               </geometry>
             </collision>

File: scout/scout_description/urdf/scout_mini_wheel_4.xacro (robot description, xacro)
@@ -59,7 +59,7 @@
                 rpy="0 0 0" />
               <geometry>
-                <mesh
-                  filename="package://scout_description/meshes/wheel.dae" />
-                  <!-- <cylinder radius="0.08" length="0.084"/> -->
+                <!-- <mesh
+                  filename="package://scout_description/meshes/wheel.dae" /> -->
+                  <cylinder radius="0.08" length="0.084"/>
               </geometry>
             </collision>
