Commit message: fix path error

File: bunker/bunker_description/urdf/bunker.xacro (robot description, xacro)
@@ -4,5 +4,5 @@
   <!-- ROS 2: use package share for mesh paths -->
   <xacro:property name="pkg_share"  value="$(find bunker_description)"/>
-  <xacro:property name="mesh_dir"   value="${pkg_share}/meshes"/>
+  <xacro:property name="mesh_dir" value="package://bunker_description/meshes"/>
   <xacro:property name="mesh_scale" value="0.001 0.001 0.001"/>
   <link name="base_link">
